File: Mainboard.sch (EAGLE design)
At the start: 68 parts, among them IC1 MS5611-01BA03, IC2 MCP73831, Q1 BSS84, U1 LM2937IMP-3.3, U2 USD-SOCKETNEW

Commit message: Fixed JTAG connector and rewired SDIO
Parts:
- removed X1: (no value), jtag:JTAG_JTAG10_2.54-SMD
- added C22: 100nF, SparkFun-Capacitors:CAP0805
- added R16, R17, R18: 47K, SparkFun-Passives:RESISTOR0805-RES
- added R19, R20, R21, R22: 100K, SparkFun-Passives:RESISTOR0805-RES
- R1, R3: value (none) -> 47K
Connections:
- removed net ADC1_IN1: STM32F401RBT6PORTA_L.PA0
- removed net ADC1_IN2: STM32F401RBT6PORTA_L.PA1
- removed net N$20: STM32F401RBT6PORTC_H.PC10, U3.INT
- removed net N$3: X1.4
- removed net N$32: U$2.RTCK
- removed net N$33: U$2.GND1
- removed net N$34: U$2.GND
- removed net N$35: U$2.VCC
- removed net N$36: U$2.TMS
- removed net N$37: U$2.TCLK
- removed net N$38: U$2.TDO
- removed net N$39: U$2.TDI
- removed net N$4: X1.2
- removed net N$40: U$2.RST
- removed net N$6: U$2.GND2
- removed net N$7: R1.2, U2.CD2
- removed net SD_MISO: R3.1, STM32F401RBT6PORTA_L.PA6, U2.DO
- removed net SD_MOSI: STM32F401RBT6PORTA_L.PA7, U2.DI
- removed net SD_NSS: STM32F401RBT6PORTA_L.PA4, U2.CS
- removed net SD_SCK: STM32F401RBT6PORTA_L.PA5, U2.SCK
- new net IMU_INT: U3.INT
- new net SDIO_CLK: STM32F401RBT6PORTC_H.PC12, U2.SCK
- new net SDIO_CMD: R1.2, STM32F401RBT6PORTD/OSC.PD2, U2.DI
- new net SDIO_D0: R17.2, STM32F401RBT6PORTC_H.PC8, U2.DO
- new net SDIO_D1: R18.2, STM32F401RBT6PORTC_H.PC9, U2.RSV
- new net SDIO_D2: R16.2, STM32F401RBT6PORTC_H.PC10, U2.NC
- new net SDIO_D3: R3.2, STM32F401RBT6PORTC_H.PC11, U2.CS
- new net SD_DETECT: STM32F401RBT6PORTC_H.PC13, U2.SHIELD@1
- net GND: now also C22.1, R19.1, U$2.GND, U$2.GND1, U$2.GND2, U2.CD1, U2.CD2; no longer R1.1, U2.SHIELD@1, X1.10, X1.8
- net GPS_SCL: now also U$5.19_SCL2
- net GPS_SDA: now also U$5.18_SDA2
- net JTCK: now also R19.2, U$2.TCLK; no longer X1.9
- net JTDI: now also R22.1, U$2.TDI; no longer X1.5
- net JTDO: now also R21.1, U$2.TDO; no longer X1.6
- net JTMS: now also R20.1, U$2.TMS; no longer X1.7
- net JTRST: now also U$2.RST; no longer X1.3
- net TIM3_CH3: now also STM32F401RBT6PORTB_L.PB0; no longer STM32F401RBT6PORTC_H.PC8
- net TIM3_CH4: now also STM32F401RBT6PORTB_L.PB1; no longer STM32F401RBT6PORTC_H.PC9
- net VDD: now also C22.2, R1.1, R16.1, R17.1, R18.1, R20.2, R21.2, R22.2, R3.1, U$2.VCC; no longer R3.2, U2.CD1, X1.1
Other:
- note added: "SD Card"
- note added: "Servo Breakouts"
- note removed: "Consider switching to SDIO but CMD is missing from 64 pin chip"
- note removed: "Switch the connector type on this to the one in Jons/matts library"
- moved on the sheet: C1, C10, C11, C12, C13, C14, C15, C16, C17, C18, C19, C2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

Commit message: Tidied board layout
Connections:
- net N$10 renamed RFM_MOSI
- net N$11 renamed RFM_RST
- net N$12 renamed RFM_DI0
- net N$2 renamed RFM_MISO
- net N$8 renamed RFM_NSS
- net N$9 renamed RFM_SCK
Other:
- note added: "GPS"
- note added: "MPU"
- note added: "Power Regulation"
- note added: "RFM Radio"
- note added: "USB and Charging"
- moved on the sheet: C1, C10, C11, C12, C13, C14, C15, C16, C17, C18, C19, C2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

Commit message: Updated schematic
Parts:
- added U$10, U$7, U$9: SERVO, b3noxley:SERVO
Changed lines of the file:
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@@
 <part name="SUPPLY2" library="supply2" deviceset="VDD" device=""/>
 <part name="C22" library="SparkFun-Capacitors" deviceset="CAP" device="0805" value="100nF"/>
+<part name="U$7" library="b3noxley" deviceset="SERVO" device=""/>
+<part name="U$9" library="b3noxley" deviceset="SERVO" device=""/>
+<part name="U$10" library="b3noxley" deviceset="SERVO" device=""/>
 </parts>
 <sheets>
@@
 <instance part="SUPPLY2" gate="G$1" x="55.88" y="218.44"/>
 <instance part="C22" gate="G$1" x="-12.7" y="200.66" rot="R180"/>
+<instance part="U$9" gate="G$1" x="381" y="152.4"/>
+<instance part="U$10" gate="G$1" x="411.48" y="152.4"/>
 </instances>
 <busses>

Commit message: Updated board design
Parts:
- removed U$10: SERVO, b3noxley:SERVO
Changed lines of the file:
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@@
 <part name="U$7" library="b3noxley" deviceset="SERVO" device=""/>
 <part name="U$9" library="b3noxley" deviceset="SERVO" device=""/>
-<part name="U$10" library="b3noxley" deviceset="SERVO" device=""/>
 </parts>
 <sheets>
@@
 <instance part="SUPPLY2" gate="G$1" x="55.88" y="218.44"/>
 <instance part="C22" gate="G$1" x="-12.7" y="200.66" rot="R180"/>
-<instance part="U$9" gate="G$1" x="381" y="152.4"/>
-<instance part="U$10" gate="G$1" x="411.48" y="152.4"/>
+<instance part="U$7" gate="G$1" x="363.22" y="149.86"/>
+<instance part="U$9" gate="G$1" x="398.78" y="149.86"/>
 </instances>
 <busses>

Commit message: Updated board and schematic, added power switch. changed connectors. Improved wing shape.
Parts:
- removed G1: BATTERY-HOLDER_11.6MM, battery:BATTERY-HOLDER_11.6MM
- removed SV1: (no value), con-lstb:MA08-1
- added JP4: (no value), SparkFun-Connectors:M08BM08B-SRSS-TB
- added S1: (no value), switch:255SB
Connections:
- removed net N$29: G1.+, U$5.22_V_BCKP
- new net N$2: C21.2, J1.+, S1.P
- net +4.1V: now also S1.S; no longer C21.2, J1.+
- net ADC1_IN10: now also JP4.6; no longer SV1.6
- net ADC1_IN11: now also JP4.5; no longer SV1.5
- net ADC1_IN12: now also JP4.4; no longer SV1.4
- net ADC1_IN13: now also JP4.3; no longer SV1.3
- net ADC1_IN14: now also JP4.2; no longer SV1.2
- net ADC1_IN15: now also JP4.1; no longer SV1.1
- net GND: now also JP4.7; no longer G1.-, SV1.7
- net VDD: now also JP4.8; no longer SV1.8
Changed lines of the file:
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@@
 <part name="U$6" library="zetex" deviceset="USBLC6-4" device=""/>
 <part name="C6" library="SparkFun-Capacitors" deviceset="CAP" device="0805" value="2.2nF"/>
-<part name="G1" library="battery" deviceset="BATTERY-HOLDER_11.6MM" device=""/>
 <part name="U$8" library="SWP" deviceset="RFM69" device=""/>
 <part name="GND14" library="supply1" deviceset="GND" device=""/>
@@
 <part name="SUPPLY12" library="supply2" deviceset="+5V" device=""/>
 <part name="C21" library="SparkFun-Capacitors" deviceset="CAP" device="0805" value="10uF"/>
-<part name="SV1" library="con-lstb" deviceset="MA08-1" device=""/>
 <part name="SUPPLY18" library="supply2" deviceset="VDD" device=""/>
 <part name="GND22" library="supply1" deviceset="GND" device=""/>
@@
 <part name="U$7" library="b3noxley" deviceset="SERVO" device=""/>
 <part name="U$9" library="b3noxley" deviceset="SERVO" device=""/>
+<part name="JP4" library="SparkFun-Connectors" deviceset="M08" device="BM08B-SRSS-TB"/>
+<part name="S1" library="switch" deviceset="255SB" device=""/>
 </parts>
 <sheets>
@@
 <text x="297.18" y="246.38" size="7.112" layer="91">GPS</text>
 <text x="78.74" y="218.44" size="7.112" layer="91">Power Regulation</text>
+<text x="325.12" y="190.5" size="1.778" layer="91">NC</text>
 </plain>
 <instances>
@@
 <instance part="U$6" gate="G$1" x="304.8" y="50.8"/>
 <instance part="C6" gate="G$1" x="419.1" y="193.04"/>
-<instance part="G1" gate="G$1" x="292.1" y="185.42" rot="R90"/>
 <instance part="U$8" gate="G$1" x="396.24" y="43.18"/>
 <instance part="GND14" gate="1" x="81.28" y="233.68"/>
@@
 <instance part="SUPPLY12" gate="+5V" x="91.44" y="213.36"/>
 <instance part="C21" gate="G$1" x="332.74" y="22.86" rot="R90"/>
-<instance part="SV1" gate="1" x="27.94" y="73.66"/>
 <instance part="SUPPLY18" gate="G$1" x="35.56" y="86.36"/>
 <instance part="GND22" gate="1" x="40.64" y="86.36" rot="R180"/>
@@
 <instance part="U$7" gate="G$1" x="363.22" y="149.86"/>
 <instance part="U$9" gate="G$1" x="398.78" y="149.86"/>
+<instance part="JP4" gate="G$1" x="27.94" y="73.66"/>
+<instance part="S1" gate="1" x="314.96" y="35.56" rot="MR270"/>
 </instances>
 <busses>
@@
 <pinref part="GND6" gate="1" pin="GND"/>
 <wire x1="325.12" y1="180.34" x2="325.12" y2="175.26" width="0.1524" layer="91"/>
-<pinref part="G1" gate="G$1" pin="-"/>
-<wire x1="325.12" y1="180.34" x2="292.1" y2="180.34" width="0.1524" layer="91"/>
 <pinref part="U$5" gate="G$1" pin="24_GND"/>
-<junction x="325.12" y="180.34"/>
 </segment>
 <segment>
@@
 </segment>
 <segment>
-<pinref part="SV1" gate="1" pin="7"/>
-<wire x1="35.56" y1="81.28" x2="40.64" y2="81.28" width="0.1524" layer="91"/>
+<wire x1="33.02" y1="81.28" x2="40.64" y2="81.28" width="0.1524" layer="91"/>
 <pinref part="GND22" gate="1" pin="GND"/>
 <wire x1="40.64" y1="81.28" x2="40.64" y2="83.82" width="0.1524" layer="91"/>
+<pinref part="JP4" gate="G$1" pin="7"/>
 </segment>
 <segment>
@@
 <wire x1="93.98" y1="12.7" x2="93.98" y2="10.16" width="0.1524" layer="91"/>
 <junction x="93.98" y="12.7"/>
-</segment>
-<segment>
-<pinref part="SV1" gate="1" pin="8"/>
-<pinref part="SUPPLY18" gate="G$1" pin="VDD"/>
 </segment>
 <segment>
@@
 <junction x="55.88" y="215.9"/>
 </segment>
+<segment>
+<pinref part="SUPPLY18" gate="G$1" pin="VDD"/>
+<pinref part="JP4" gate="G$1" pin="8"/>
+<wire x1="33.02" y1="83.82" x2="35.56" y2="83.82" width="0.1524" layer="91"/>
+</segment>
 </net>
 <net name="JTRST" class="0">
@@
 </segment>
 </net>
-<net name="N$29" class="0">
-<segment>
-<pinref part="G1" gate="G$1" pin="+"/>
-<pinref part="U$5" gate="G$1" pin="22_V_BCKP"/>
-<wire x1="292.1" y1="190.5" x2="325.12" y2="190.5" width="0.1524" layer="91"/>
-</segment>
-</net>
 <net name="USART1_TX" class="0">
 <segment>
@@
 <segment>
 <pinref part="IC2" gate="G$1" pin="VBAT"/>
-<wire x1="325.12" y1="33.02" x2="322.58" y2="33.02" width="0.1524" layer="91"/>
-<pinref part="J1" gate="G$1" pin="+"/>
 <pinref part="SUPPLY16" gate="P" pin="+4.1V"/>
-<wire x1="322.58" y1="33.02" x2="307.34" y2="33.02" width="0.1524" layer="91"/>
+<wire x1="307.34" y1="33.02" x2="307.34" y2="35.56" width="0.1524" layer="91"/>
 <wire x1="307.34" y1="33.02" x2="304.8" y2="33.02" width="0.1524" layer="91"/>
-<wire x1="307.34" y1="33.02" x2="307.34" y2="35.56" width="0.1524" layer="91"/>
-<wire x1="322.58" y1="33.02" x2="322.58" y2="30.48" width="0.1524" layer="91"/>
-<pinref part="C21" gate="G$1" pin="2"/>
-<wire x1="322.58" y1="30.48" x2="335.28" y2="30.48" width="0.1524" layer="91"/>
-<wire x1="335.28" y1="30.48" x2="335.28" y2="22.86" width="0.1524" layer="91"/>
-<junction x="322.58" y="33.02"/>
+<pinref part="S1" gate="1" pin="S"/>
+<wire x1="309.88" y1="30.48" x2="307.34" y2="30.48" width="0.1524" layer="91"/>
+<wire x1="307.34" y1="30.48" x2="307.34" y2="33.02" width="0.1524" layer="91"/>
+<junction x="307.34" y="33.02"/>
 </segment>
 <segment>
@@
 <segment>
 <pinref part="STM32F401RBT6" gate="PORTC_L" pin="PC0"/>
-<wire x1="48.26" y1="78.74" x2="35.56" y2="78.74" width="0.1524" layer="91"/>
+<wire x1="48.26" y1="78.74" x2="33.02" y2="78.74" width="0.1524" layer="91"/>
 <label x="35.56" y="78.74" size="1.778" layer="95"/>
-<pinref part="SV1" gate="1" pin="6"/>
+<pinref part="JP4" gate="G$1" pin="6"/>
 </segment>
 </net>
@@
 <segment>
 <pinref part="STM32F401RBT6" gate="PORTC_L" pin="PC1"/>
-<wire x1="48.26" y1="76.2" x2="35.56" y2="76.2" width="0.1524" layer="91"/>
+<wire x1="48.26" y1="76.2" x2="33.02" y2="76.2" width="0.1524" layer="91"/>
 <label x="35.56" y="76.2" size="1.778" layer="95"/>
-<pinref part="SV1" gate="1" pin="5"/>
+<pinref part="JP4" gate="G$1" pin="5"/>
 </segment>
 </net>
@@
 <segment>
 <pinref part="STM32F401RBT6" gate="PORTC_L" pin="PC2"/>
-<wire x1="48.26" y1="73.66" x2="35.56" y2="73.66" width="0.1524" layer="91"/>
+<wire x1="48.26" y1="73.66" x2="33.02" y2="73.66" width="0.1524" layer="91"/>
 <label x="35.56" y="73.66" size="1.778" layer="95"/>
-<pinref part="SV1" gate="1" pin="4"/>
+<pinref part="JP4" gate="G$1" pin="4"/>
 </segment>
 </net>
@@
 <segment>
 <pinref part="STM32F401RBT6" gate="PORTC_L" pin="PC3"/>
-<wire x1="48.26" y1="71.12" x2="35.56" y2="71.12" width="0.1524" layer="91"/>
+<wire x1="48.26" y1="71.12" x2="33.02" y2="71.12" width="0.1524" layer="91"/>
 <label x="35.56" y="71.12" size="1.778" layer="95"/>
-<pinref part="SV1" gate="1" pin="3"/>
+<pinref part="JP4" gate="G$1" pin="3"/>
 </segment>
 </net>
@@
 <segment>
 <pinref part="STM32F401RBT6" gate="PORTC_L" pin="PC4"/>
-<wire x1="48.26" y1="68.58" x2="35.56" y2="68.58" width="0.1524" layer="91"/>
+<wire x1="48.26" y1="68.58" x2="33.02" y2="68.58" width="0.1524" layer="91"/>
 <label x="35.56" y="68.58" size="1.778" layer="95"/>
-<pinref part="SV1" gate="1" pin="2"/>
+<pinref part="JP4" gate="G$1" pin="2"/>
 </segment>
 </net>
@@
 <segment>
 <pinref part="STM32F401RBT6" gate="PORTC_L" pin="PC5"/>
-<wire x1="48.26" y1="66.04" x2="35.56" y2="66.04" width="0.1524" layer="91"/>
+<wire x1="48.26" y1="66.04" x2="33.02" y2="66.04" width="0.1524" layer="91"/>
 <label x="35.56" y="66.04" size="1.778" layer="95"/>
-<pinref part="SV1" gate="1" pin="1"/>
+<pinref part="JP4" gate="G$1" pin="1"/>
 </segment>
 </net>
@@
 </segment>
 </net>
+<net name="N$2" class="0">
+<segment>
+<wire x1="325.12" y1="33.02" x2="322.58" y2="33.02" width="0.1524" layer="91"/>
+<pinref part="J1" gate="G$1" pin="+"/>
+<wire x1="322.58" y1="33.02" x2="322.58" y2="30.48" width="0.1524" layer="91"/>
+<pinref part="C21" gate="G$1" pin="2"/>
+<wire x1="322.58" y1="30.48" x2="335.28" y2="30.48" width="0.1524" layer="91"/>
+<wire x1="335.28" y1="30.48" x2="335.28" y2="22.86" width="0.1524" layer="91"/>
+<pinref part="S1" gate="1" pin="P"/>
+<wire x1="320.04" y1="33.02" x2="322.58" y2="33.02" width="0.1524" layer="91"/>
+<junction x="322.58" y="33.02"/>
+</segment>
+</net>

Commit message: Started wiring board
Parts:
- renumbered C1 to C1_MPU_10, C10 to C10_LM2937_3, C11 to C11_LM2937_3, C12 to C12_RFM69_8, C13 to C13_RFM69_8, C14 to C14_RFM69_1, C15 to C15_MS5611_1, C16 to C16_STM32_13, C17 to C17_STM32_32, C18 to C18_STM32_48, C19 to C19_STM32_64, C2 to C2_MPU_20, C20 to C20_STM32_19, C21 to C21_MCP73831_VSS, C22 to C22_JTAG_VCC, C3 to C3_MPU_3, C4 to C4_MCP73831_4, C5 to C5_MCP73831_4, C6 to C6_USB_VBUS, C7 to C7_RESET_DEBOUNCE, C8 to C8_LM2937_1, C9 to C9_LM2937_1
